File: Project.kicad_sch (KiCad schematic)
At the start: 0 parts

Commit message: Added 2 motor drivers and a sensor UC
Parts:
- added U1, U2: DRV8833PW, Package_SO:TSSOP-16_4.4x5mm_P0.65mm, symbol Driver_Motor:DRV8833PW
- added U3: INA219AxD, Package_SO:SOIC-8_3.9x4.9mm_P1.27mm, symbol Sensor_Energy:INA219AxD
Changed lines of the file:
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@@
     (comment 2 "Author 1: Branden Nkhahle (NKHTLO001)")
+  )
+  (symbol (lib_id "Driver_Motor:DRV8833PW") (at 134.62 55.88 0) (unit 1)
+    (in_bom yes) (on_board yes) (dnp no) (fields_autoplaced)
+    (property "Reference" "U2" (at 136.8141 71.12 0)
+      (effects (font (size 1.27 1.27)) (justify left))
+    )
+    (property "Value" "DRV8833PW" (at 136.8141 73.66 0)
+      (effects (font (size 1.27 1.27)) (justify left))
+    )
+    (property "Footprint" "Package_SO:TSSOP-16_4.4x5mm_P0.65mm" (at 146.05 44.45 0)
+      (effects (font (size 1.27 1.27)) (justify left) hide)
+    )
+    (property "Datasheet" "http://www.ti.com/lit/ds/symlink/drv8833.pdf" (at 130.81 41.91 0)
+      (effects (font (size 1.27 1.27)) hide)
+    )
+    (pin "4")
+    (pin "12")
+    (pin "8")
+    (pin "16")
+    (pin "1")
+    (pin "6")
+    (pin "2")
+    (pin "10")
+    (pin "11")
+    (pin "15")
+    (pin "14")
+    (pin "5")
+    (pin "3")
+    (pin "7")
+    (pin "9")
+    (pin "13")
+    (instances
+      (project "Project"
+        (path "/17758c82-f715-4af2-8495-50ca19713f99"
+          (reference "U2") (unit 1)
+        )
+      )
+    )
+  )
+  (symbol (lib_id "Sensor_Energy:INA219AxD") (at 170.18 52.07 0) (unit 1)
+    (in_bom yes) (on_board yes) (dnp no) (fields_autoplaced)
+    (property "Reference" "U3" (at 172.3741 39.37 0)
+      (effects (font (size 1.27 1.27)) (justify left))
+    )
+    (property "Value" "INA219AxD" (at 172.3741 41.91 0)
+      (effects (font (size 1.27 1.27)) (justify left))
+    )
+    (property "Footprint" "Package_SO:SOIC-8_3.9x4.9mm_P1.27mm" (at 190.5 60.96 0)
+      (effects (font (size 1.27 1.27)) hide)
+    )
+    (property "Datasheet" "http://www.ti.com/lit/ds/symlink/ina219.pdf" (at 179.07 54.61 0)
+      (effects (font (size 1.27 1.27)) hide)
+    )
+    (pin "5")
+    (pin "2")
+    (pin "6")
+    (pin "1")
+    (pin "7")
+    (pin "8")
+    (pin "3")
+    (pin "4")
+    (instances
+      (project "Project"
+        (path "/17758c82-f715-4af2-8495-50ca19713f99"
+          (reference "U3") (unit 1)
+        )
+      )
+    )
+  )
+  (symbol (lib_id "Driver_Motor:DRV8833PW") (at 80.01 55.88 0) (unit 1)
+    (in_bom yes) (on_board yes) (dnp no) (fields_autoplaced)
+    (property "Reference" "U1" (at 82.2041 71.12 0)
+      (effects (font (size 1.27 1.27)) (justify left))
+    )
+    (property "Value" "DRV8833PW" (at 82.2041 73.66 0)
+      (effects (font (size 1.27 1.27)) (justify left))
+    )
+    (property "Footprint" "Package_SO:TSSOP-16_4.4x5mm_P0.65mm" (at 91.44 44.45 0)
+      (effects (font (size 1.27 1.27)) (justify left) hide)
+    )
+    (property "Datasheet" "http://www.ti.com/lit/ds/symlink/drv8833.pdf" (at 76.2 41.91 0)
+      (effects (font (size 1.27 1.27)) hide)
+    )
+    (pin "12")
+    (pin "3")
+    (pin "4")
+    (pin "2")
+    (pin "5")
+    (pin "7")
+    (pin "10")
+    (pin "8")
+    (pin "1")
+    (pin "6")
+    (pin "15")
+    (pin "11")
+    (pin "16")
+    (pin "9")
+    (pin "14")
+    (pin "13")
+    (instances
+      (project "Project"
+        (path "/17758c82-f715-4af2-8495-50ca19713f99"
+          (reference "U1") (unit 1)
+        )
+      )
+    )
   )
   (sheet_instances
